Commit message: working for cube and cuboid

File: ur5_gripper_description/urdf/ur5_gripper.urdf (robot description, URDF)
Before this commit: robot ur5_gripper, 26 links, 25 joints
Joints:
- joint robotiq_finger_1_joint_1: limit lower=0.0495 upper=1.2218 effort=100 velocity=100 -> lower=0.0495 upper=1.2218 effort=70 velocity=100
- joint robotiq_finger_1_joint_2: limit lower=0.0 upper=1.5708 effort=100 velocity=100 -> lower=0.0 upper=1.5708 effort=70 velocity=100
- joint robotiq_finger_1_joint_3: limit lower=-1.2217 upper=-0.0523 effort=100 velocity=100 -> lower=-1.2217 upper=-0.0523 effort=70 velocity=100
- joint robotiq_finger_2_joint_1: limit lower=0.0495 upper=1.2218 effort=100 velocity=100 -> lower=0.0495 upper=1.2218 effort=70 velocity=100
- joint robotiq_finger_2_joint_2: limit lower=0.0 upper=1.5708 effort=100 velocity=100 -> lower=0.0 upper=1.5708 effort=70 velocity=100
- joint robotiq_finger_2_joint_3: limit lower=-1.2217 upper=-0.0523 effort=100 velocity=100 -> lower=-1.2217 upper=-0.0523 effort=70 velocity=100
- joint robotiq_finger_middle_joint_1: limit lower=0.0495 upper=1.2218 effort=100 velocity=100 -> lower=0.0495 upper=1.2218 effort=70 velocity=100
- joint robotiq_finger_middle_joint_2: limit lower=0.0 upper=1.5708 effort=100 velocity=100 -> lower=0.0 upper=1.5708 effort=70 velocity=100
- joint robotiq_finger_middle_joint_3: limit lower=-1.2217 upper=-0.0523 effort=100 velocity=100 -> lower=-1.2217 upper=-0.0523 effort=70 velocity=100
- joint robotiq_palm_finger_1_joint: limit lower=-0.1784 upper=0.192 effort=100 velocity=100 -> lower=-0.1784 upper=0.192 effort=70 velocity=100
- joint robotiq_palm_finger_2_joint: limit lower=-0.192 upper=0.1784 effort=100 velocity=100 -> lower=-0.192 upper=0.1784 effort=70 velocity=100
